File: kicad/choc/tackle-choc.kicad_pcb (KiCad board)
At the start: 2 copper layers, 158 x 119 mm, 114 parts, among them J1 Conn_01x02, SW1 SW_Push, SW10 SW_Push, SW11 SW_Push, SW12 SW_Push, SW13 SW_Push, SW14 SW_Push, SW15 SW_Push, SW16 SW_Push, SW17 SW_Push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

Commit message: 1.1 - widen cutouts to make sawing PCBs easier
Other:
- outline, holes or cut-outs redrawn
- board text added: "tackle 1.1"
- board text removed: "tackle 1.0"
