File: kicad/choc/tackle-choc.kicad_sch (KiCad schematic)
At the start: 114 parts, among them J1 Conn_01x02, SW1 SW_Push, SW10 SW_Push, SW11 SW_Push, SW12 SW_Push, SW13 SW_Push, SW14 SW_Push, SW15 SW_Push, SW16 SW_Push, SW17 SW_Push, SW18 SW_Push, SW19 SW_Push, SW2 SW_Push, SW20 SW_Push, SW21 SW_Push, SW22 SW_Push, SW23 SW_Push, SW24 SW_Push, SW25 SW_Push, SW26 SW_Push, SW27 SW_Push, SW28 SW_Push, SW29 SW_Push, SW3 SW_Push, SW30 SW_Push, SW31 SW_Push, SW32 SW_Push, SW33 SW_Push, SW34 SW_Push, SW35 SW_Push, SW36 SW_Push, SW37 SW_Push, SW38 SW_Push, SW39 SW_Push, SW4 SW_Push, SW40 SW_Push, SW41 SW_Push, SW42 SW_Push, SW43 SW_Push, SW44 SW_Push, SW45 SW_Push, SW46 SW_Push, SW47 SW_Push, SW48 SW_Push, SW5 SW_Push, SW6 SW_Push, SW7 SW_Push, SW8 SW_Push, SW9 SW_Push, U1 nice!nano

Commit message: Swap power switch direction, update fabrication settings
Parts:
- LOGO1, LOGO2: now left out of the parts list
Changed lines of the file:
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@@
 		(unit 1)
 		(exclude_from_sim no)
-		(in_bom yes)
+		(in_bom no)
 		(on_board yes)
 		(dnp no)
@@
 		(unit 1)
 		(exclude_from_sim no)
-		(in_bom yes)
+		(in_bom no)
 		(on_board yes)
 		(dnp no)

Commit message: Adjust strap slot sizes
Connections:
- net RAW: now also SPDT1.3 (C); no longer SPDT1.1 (A)
Changed lines of the file:
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@@
-	)
-	(no_connect
-		(at 248.92 129.54)
 	)
 	(no_connect
@@
 	(no_connect
 		(at 264.16 80.01)
+	)
+	(no_connect
+		(at 248.92 124.46)
 	)
 	(no_connect
@@
 	(global_label "RAW"
 		(shape input)
-		(at 248.92 124.46 0)
+		(at 248.92 129.54 0)
 		(fields_autoplaced yes)
 		(effects
@@
 		)
 		(property "Intersheetrefs" "${INTERSHEET_REFS}"
-			(at 255.061 124.46 0)
-			(effects
-				(font
+			(at 255.061 129.54 0)
+			(effects
+				(font
